File: parrot_imu.kicad_sch (KiCad schematic)
At the start: 17 parts

Commit message: design review with tony
Connections:
- net +3.3V: no longer U?.15 (3V3), U?.46 (3V3)
Other:
- note added: "Add board mount xt30 connection to stop cookage"
- note added: "TVS Diode for protection SMAJ24AQ-13-F?"
- note added: "TVS Diodes (PEDISCAN)"
- note removed: "Shottkey Diode for protection?"
Changed lines of the file:
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@@
-    (stroke (width 0) (type default) (color 0 0 0 0))
-  )
-  (wire (pts (xy 226.06 134.62) (xy 236.22 134.62))
     (stroke (width 0) (type default) (color 0 0 0 0))
   )
@@
   )
   (wire (pts (xy 332.74 82.55) (xy 332.74 91.44))
-    (stroke (width 0) (type default) (color 0 0 0 0))
-  )
-  (wire (pts (xy 154.94 165.1) (xy 170.18 165.1))
     (stroke (width 0) (type default) (color 0 0 0 0))
   )
@@
     (effects (font (size 1.27 1.27)) (justify left bottom))
   )
+  (text "TVS Diodes (PEDISCAN)\n" (at 344.17 66.04 0)
+    (effects (font (size 1.27 1.27)) (justify left bottom))
+  )
   (text "Do I need to chuck on a couple of diodes or something here like with older teensies?"
     (at 162.56 116.84 0)
@@
     (effects (font (size 1.27 1.27)) (justify left bottom))
   )
-  (text "Shottkey Diode for protection?" (at 21.59 110.49 0)
+  (text "TVS Diode for protection SMAJ24AQ-13-F?" (at 21.59 110.49 0)
+    (effects (font (size 1.27 1.27)) (justify left bottom))
+  )
+  (text "Add board mount xt30 connection to stop cookage" (at 16.51 104.14 0)
     (effects (font (size 1.27 1.27)) (justify left bottom))
   )
@@
   (label "Eth_tx-" (at 226.06 201.93 0)
     (effects (font (size 1.27 1.27)) (justify left bottom))
-  )
-  (symbol (lib_id "power:+3.3V") (at 236.22 134.62 0) (unit 1)
-    (in_bom yes) (on_board yes) (fields_autoplaced)
-    (property "Reference" "#PWR?" (id 0) (at 236.22 138.43 0)
-      (effects (font (size 1.27 1.27)) hide)
-    )
-    (property "Value" "+3.3V" (id 1) (at 236.22 129.54 0))
-    (property "Footprint" "" (id 2) (at 236.22 134.62 0)
-      (effects (font (size 1.27 1.27)) hide)
-    )
-    (property "Datasheet" "" (id 3) (at 236.22 134.62 0)
-      (effects (font (size 1.27 1.27)) hide)
-    )
-    (pin "1")
   )
   (symbol (lib_id "Device:C") (at 313.69 100.33 0) (unit 1)
@@
     )
     (property "Datasheet" "" (id 3) (at 325.12 96.52 0)
-      (effects (font (size 1.27 1.27)) hide)
-    )
-    (pin "1")
-  )
-  (symbol (lib_id "power:+3.3V") (at 154.94 165.1 0) (unit 1)
-    (in_bom yes) (on_board yes) (fields_autoplaced)
-    (property "Reference" "#PWR?" (id 0) (at 154.94 168.91 0)
-      (effects (font (size 1.27 1.27)) hide)
-    )
-    (property "Value" "+3.3V" (id 1) (at 154.94 160.02 0))
-    (property "Footprint" "" (id 2) (at 154.94 165.1 0)
-      (effects (font (size 1.27 1.27)) hide)
-    )
-    (property "Datasheet" "" (id 3) (at 154.94 165.1 0)
       (effects (font (size 1.27 1.27)) hide)
     )
@@
   )
   (symbol_instances
-    (path "/0f2fa5a7-2f21-4ddc-bd16-0af5047c701f"
-      (reference "#PWR?") (unit 1) (value "+3.3V") (footprint "")
-    )
     (path "/21bc302e-37b5-4465-b524-2fb59916f8c8"
       (reference "#PWR?") (unit 1) (value "+3.3V") (footprint "")
@@
       (reference "#PWR?") (unit 1) (value "+3.3V") (footprint "")
     )
-    (path "/564be391-f282-4047-8b76-1b3d14e61008"
-      (reference "#PWR?") (unit 1) (value "+3.3V") (footprint "")
-    )
