File: parrot_imu.kicad_sch (KiCad schematic)
At the start: 29 parts, among them J1 Conn_01x02_Male, J2 SI-60062-F, J3 TB005-762-02BE, U1 TR05S3V3, U2 VR10S05, U3 Spark_fun_ICM-20948, U4 Teensy4.1, U5 TJA1441AT/0Z, U6 ESDCAN24-2BLY

Commit message: dump of progress
Parts:
- J1: footprint Connector_AMASS:AMASS_XT30PW-F_1x02_P2.50mm_Horizontal -> Connector_AMASS:AMASS_XT30PW-M_1x02_P2.50mm_Horizontal
Connections:
- net Can_rx: now also U4.22 (30_CRX3); no longer U4.45 (23_A9_CRX1_MCLK1)
- net Can_tx: now also U4.23 (31_CTX3); no longer U4.44 (22_A8_CTX1)
Changed lines of the file:
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@@
   (no_connect (at 170.18 195.58))
   (no_connect (at 170.18 207.01))
-  (no_connect (at 170.18 182.88))
+  (no_connect (at 226.06 139.7))
   (no_connect (at 190.5 217.17))
   (no_connect (at 170.18 147.32))
@@
   (no_connect (at 170.18 154.94))
   (no_connect (at 226.06 170.18))
+  (no_connect (at 226.06 137.16))
   (no_connect (at 226.06 177.8))
   (no_connect (at 170.18 199.39))
@@
   (no_connect (at 170.18 137.16))
   (no_connect (at 194.31 217.17))
-  (no_connect (at 170.18 185.42))
   (no_connect (at 226.06 160.02))
   (no_connect (at 170.18 201.93))
@@
     (stroke (width 0) (type default) (color 0 0 0 0))
   )
+  (wire (pts (xy 157.48 182.88) (xy 170.18 182.88))
+    (stroke (width 0) (type default) (color 0 0 0 0))
+  )
   (wire (pts (xy 256.54 57.15) (xy 264.16 57.15))
     (stroke (width 0) (type default) (color 0 0 0 0))
@@
     (stroke (width 0) (type default) (color 0 0 0 0))
   )
-  (wire (pts (xy 227.33 137.16) (xy 226.06 137.16))
-    (stroke (width 0) (type default) (color 0 0 0 0))
-  )
   (wire (pts (xy 180.34 97.79) (xy 186.69 97.79))
     (stroke (width 0) (type default) (color 0 0 0 0))
@@
     (stroke (width 0) (type default) (color 0 0 0 0))
   )
-  (wire (pts (xy 227.33 139.7) (xy 226.06 139.7))
-    (stroke (width 0) (type default) (color 0 0 0 0))
-  )
   (wire (pts (xy 360.68 71.12) (xy 372.11 71.12))
     (stroke (width 0) (type default) (color 0 0 0 0))
@@
     (stroke (width 0) (type default) (color 0 0 0 0))
   )
+  (wire (pts (xy 157.48 185.42) (xy 170.18 185.42))
+    (stroke (width 0) (type default) (color 0 0 0 0))
+  )
   (wire (pts (xy 81.28 156.21) (xy 72.39 156.21))
     (stroke (width 0) (type default) (color 0 0 0 0))
@@
     (effects (font (size 1.27 1.27)) (justify left bottom))
   )
-  (label "Can_rx" (at 227.33 137.16 0)
-    (effects (font (size 1.27 1.27)) (justify left bottom))
-  )
-  (label "Can_tx" (at 227.33 139.7 0)
+  (label "Can_rx" (at 157.48 182.88 0)
+    (effects (font (size 1.27 1.27)) (justify left bottom))
+  )
+  (label "Can_tx" (at 157.48 185.42 0)
     (effects (font (size 1.27 1.27)) (justify left bottom))
   )
@@
       (effects (font (size 1.27 1.27)) (justify right))
     )
-    (property "Footprint" "Connector_AMASS:AMASS_XT30PW-F_1x02_P2.50mm_Horizontal" (id 2) (at 34.29 129.54 0)
+    (property "Footprint" "Connector_AMASS:AMASS_XT30PW-M_1x02_P2.50mm_Horizontal" (id 2) (at 34.29 129.54 0)
       (effects (font (size 1.27 1.27)) hide)
     )
@@
     )
     (path "/35ca6dd5-0fe6-4149-b1eb-072213388a9c"
-      (reference "J1") (unit 1) (value "Conn_01x02_Male") (footprint "Connector_AMASS:AMASS_XT30PW-F_1x02_P2.50mm_Horizontal")
+      (reference "J1") (unit 1) (value "Conn_01x02_Male") (footprint "Connector_AMASS:AMASS_XT30PW-M_1x02_P2.50mm_Horizontal")
     )
     (path "/0d20f8ee-a6f7-49a8-87a9-065aa3be88a2"

Commit message: pcb redesign
Connections:
- net GND: no longer J2.5 (RCT)
- net at C6.1, J2.2 (TCT): now also J2.5 (RCT)
Other:
- moved on the sheet: C6
Changed lines of the file:
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@@
   (junction (at 304.8 68.58) (diameter 0) (color 0 0 0 0)
   )
-  (junction (at 279.4 158.75) (diameter 0) (color 0 0 0 0)
+  (junction (at 290.83 156.21) (diameter 0) (color 0 0 0 0)
   )
   (junction (at 52.07 127) (diameter 0) (color 0 0 0 0)
@@
     (stroke (width 0) (type default) (color 0 0 0 0))
   )
+  (wire (pts (xy 290.83 158.75) (xy 290.83 156.21))
+    (stroke (width 0) (type default) (color 0 0 0 0))
+  )
   (wire (pts (xy 256.54 57.15) (xy 264.16 57.15))
     (stroke (width 0) (type default) (color 0 0 0 0))
@@
     (stroke (width 0) (type default) (color 0 0 0 0))
   )
-  (wire (pts (xy 279.4 158.75) (xy 300.99 158.75))
-    (stroke (width 0) (type default) (color 0 0 0 0))
-  )
   (wire (pts (xy 226.06 165.1) (xy 231.14 165.1))
     (stroke (width 0) (type default) (color 0 0 0 0))
@@
     (stroke (width 0) (type default) (color 0 0 0 0))
   )
+  (wire (pts (xy 300.99 158.75) (xy 290.83 158.75))
+    (stroke (width 0) (type default) (color 0 0 0 0))
+  )
   (wire (pts (xy 180.34 100.33) (xy 186.69 100.33))
     (stroke (width 0) (type default) (color 0 0 0 0))
@@
     (stroke (width 0) (type default) (color 0 0 0 0))
   )
+  (wire (pts (xy 290.83 151.13) (xy 300.99 151.13))
+    (stroke (width 0) (type default) (color 0 0 0 0))
+  )
+  (wire (pts (xy 279.4 156.21) (xy 290.83 156.21))
+    (stroke (width 0) (type default) (color 0 0 0 0))
+  )
   (wire (pts (xy 255.27 43.18) (xy 242.57 43.18))
     (stroke (width 0) (type default) (color 0 0 0 0))
@@
     (stroke (width 0) (type default) (color 0 0 0 0))
   )
-  (wire (pts (xy 279.4 163.83) (xy 279.4 158.75))
-    (stroke (width 0) (type default) (color 0 0 0 0))
-  )
   (wire (pts (xy 304.8 41.91) (xy 304.8 53.34))
     (stroke (width 0) (type default) (color 0 0 0 0))
   )
+  (wire (pts (xy 290.83 156.21) (xy 290.83 151.13))
+    (stroke (width 0) (type default) (color 0 0 0 0))
+  )
   (wire (pts (xy 180.34 95.25) (xy 186.69 95.25))
     (stroke (width 0) (type default) (color 0 0 0 0))
@@
   )
   (wire (pts (xy 92.71 156.21) (xy 81.28 156.21))
-    (stroke (width 0) (type default) (color 0 0 0 0))
-  )
-  (wire (pts (xy 279.4 151.13) (xy 300.99 151.13))
     (stroke (width 0) (type default) (color 0 0 0 0))
   )
@@
     (pin "1")
   )
-  (symbol (lib_id "Device:C") (at 279.4 154.94 0) (unit 1)
-    (in_bom yes) (on_board yes) (fields_autoplaced)
-    (property "Reference" "C6" (id 0) (at 283.21 153.6699 0)
+  (symbol (lib_id "Device:C") (at 279.4 160.02 0) (unit 1)
+    (in_bom yes) (on_board yes) (fields_autoplaced)
+    (property "Reference" "C6" (id 0) (at 283.21 158.7499 0)
       (effects (font (size 1.27 1.27)) (justify left))
     )
-    (property "Value" "0.1uF" (id 1) (at 283.21 156.2099 0)
+    (property "Value" "0.1uF" (id 1) (at 283.21 161.2899 0)
       (effects (font (size 1.27 1.27)) (justify left))
     )
-    (property "Footprint" "Capacitor_SMD:C_0603_1608Metric" (id 2) (at 280.3652 158.75 0)
-      (effects (font (size 1.27 1.27)) hide)
-    )
-    (property "Datasheet" "~" (id 3) (at 279.4 154.94 0)
-      (effects (font (size 1.27 1.27)) hide)
-    )
-    (property "Digikey" "1276-1935-1-ND" (id 4) (at 279.4 154.94 0)
-      (effects (font (size 1.27 1.27)) hide)
-    )
+    (property "Footprint" "Capacitor_SMD:C_0603_1608Metric" (id 2) (at 280.3652 163.83 0)
+      (effects (font (size 1.27 1.27)) hide)
+    )
+    (property "Datasheet" "~" (id 3) (at 279.4 160.02 0)
+      (effects (font (size 1.27 1.27)) hide)
+    )
+    (property "Digikey" "1276-1935-1-ND" (id 4) (at 279.4 160.02 0)
+      (effects (font (size 1.27 1.27)) hide)
+    )

Commit message: update pcb
Other:
- note added: "+24 in"
- note added: "CAN Interface"
- note added: "Ethernet"
- note added: "IMU"
- note added: "Mechanical Interface"
- note added: "Power Supply"
- note added: "Teensy"
- note removed: "Need to ad small pins to bom for ethernet"
- note removed: "This might need to be switched to i2c"
- moved on the sheet: C5, C6, C7, J2, J3, R4, R5, U3, U5, U6
