File: parrot_imu.kicad_pcb (KiCad board)
At the start: 2 copper layers, 50 x 100 mm, 29 parts, among them J1 Conn_01x02_Male, J2 SI-60062-F, J3 TB005-762-02BE, U1 TR05S3V3, U2 VR10S05, U3 Spark_fun_ICM-20948, U4 Teensy4.1, U5 TJA1441AT/0Z, U6 ESDCAN24-2BLY

Commit message: pcb redesign
Parts:
- U6: value ESDCAN24-2BLY -> SOT_24-2BLY_STM
- moved D4 11.2 mm to (87.9, 126.9), turned to 180 degrees
- moved R3 8.01 mm to (84.7, 126.8)
- moved C3 6.98 mm to (76.3, 128.3), turned to 0 degrees
- moved C6 2.52 mm to (75.8, 100.3)
- moved C7 0.30 mm to (78.5, 118.3)
Connections:
- J2 pad 5: GND -> Net-(C6-Pad1)
Routing:
- net /Eth_led: track 0.00 -> 69.2 mm
- net /Eth_tx-: track 0.00 -> 55.1 mm
- net /Eth_tx+: track 0.00 -> 54.8 mm
- net /Eth_rx+: track 0.00 -> 31.9 mm
- net /Eth_rx-: track 0.00 -> 31.8 mm
- net GND: track 48.5 -> 27.9 mm, vias 9 -> 16
- net Net-(C6-Pad1): track 4.51 -> 8.45 mm
- net +5V: track 162.9 -> 166.5 mm
- net /CS: track 27.1 -> 29.6 mm
- net +3.3V: track 7.34 -> 9.36 mm
- net /SCK: track 67.2 -> 68.9 mm
- net /MISO: track 30.6 -> 32.0 mm
- net /MOSI: track 65.5 -> 66.1 mm
- added copper zone on F.Cu, net GND
